File: hardware/beat-4.kicad_pcb (KiCad board)
At the start: 4 copper layers, 70 x 70 mm, 109 parts, among them J1001 SJ2-25404B-SMT-TR, J101 Cortex, J102 DX07S016JA3, J201 DX07S016JA3, J202 KitProg3, J401 WAGO 2601-1101, J402 WAGO 2601-1101, J403 WAGO 2601-1101, J404 WAGO 2601-1101, J405 WAGO 2601-1101, J406 WAGO 2601-1101, J407 WAGO 2601-1101, J408 WAGO 2601-1101, Q201 BSC010N04LS, Q202 BSC010N04LS, Q601 BSC010N04LS, Q701 BSC010N04LS, Q801 BSC010N04LS, Q901 BSC010N04LS, SW101 SKSG, SW102 SKSG, U1001 TLP2361, U101 ATSAMD51G, U102 TPS78433QWDRBRQ1, U201 CYPM1311-48LDXI, U301 TPSM33620S5QRDNRQ1, U501 BTT6010, Y101 32k768

Commit message: Rename
Connections:
- net /PowerDelivery/+VBUS renamed /Power USB/+VBUS
- net /PowerDelivery/+VCORE renamed /Power USB/+VCORE
- net /PowerDelivery/+VSYS renamed /Power USB/+VSYS
- net /PowerDelivery/Drain renamed /Power USB/Drain
- net /PowerDelivery/LED-Red renamed /Power USB/LED-Red
- net /PowerDelivery/RESET renamed /Power USB/RESET
- net /PowerDelivery/Rail-Input renamed /Power USB/Rail-Input
- net /PowerDelivery/Rail-Output renamed /Power USB/Rail-Output
- net /PowerDelivery/SCL renamed /Power USB/SCL
- net /PowerDelivery/SDA renamed /Power USB/SDA
- net /PowerDelivery/SWCLK renamed /Power USB/SWCLK
- net /PowerDelivery/SWDIO renamed /Power USB/SWDIO
- net /PowerDelivery/Shield renamed /Power USB/Shield
- net /PowerDelivery/USB+ renamed /Power USB/USB+
- net /PowerDelivery/USB- renamed /Power USB/USB-
- net /PowerDelivery/USB-CC1 renamed /Power USB/USB-CC1
- net /PowerDelivery/USB-CC2 renamed /Power USB/USB-CC2

Commit message: Move parts away from edge
Parts:
- moved C1001 14.7 mm to (162.0, 55.2), turned to 180 degrees
- moved U1001 10.8 mm to (162.0, 61.5)
- moved R1001 9.26 mm to (163.2, 56.8), turned to 180 degrees
- moved C1002 9.09 mm to (165.0, 63.0)
- moved D1001 6.71 mm to (160.8, 56.8), turned to 180 degrees
- moved ICON101 0.50 mm to (177.5, 58.8)
- moved ICON102 0.50 mm to (180.2, 62.5)
Connections:
- net Net-(D1001-K) renamed /MIDI In/LED
Routing:
- net /MIDI-In: track 29.8 -> 18.5 mm
- net /MIDI In/Tip: track 21.4 -> 16.5 mm
- net /MIDI In/Ring: track 7.61 -> 2.72 mm
- net +3V3: track 197.0 -> 192.5 mm
- net /MIDI In/LED: track 5.64 -> 3.24 mm
