File: hardware/PWM.kicad_sch (KiCad schematic)
At the start: 8 parts, among them J401 WAGO 2601-1101, J402 WAGO 2601-1101, J403 WAGO 2601-1101, J404 WAGO 2601-1101, J405 WAGO 2601-1101, J406 WAGO 2601-1101, J407 WAGO 2601-1101, J408 WAGO 2601-1101

Commit message: Rename
Other:
- sheet PWM 1: file PWMChannel.kicad_sch -> PWM-Channel.kicad_sch
- sheet PWM 2: file PWMChannel.kicad_sch -> PWM-Channel.kicad_sch
- sheet PWM 3: file PWMChannel.kicad_sch -> PWM-Channel.kicad_sch
- sheet PWM 4: file PWMChannel.kicad_sch -> PWM-Channel.kicad_sch
- sheet PWM Power: file PowerSwitch.kicad_sch -> Power-Switch.kicad_sch
Changed lines of the file:
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@@
 	(title_block
 		(title "V2 beat")
-		(date "2026-08-29")
+		(date "2026-08-30")
 		(rev "2026-08-29")
 		(company "Versio Duo")
@@
 			)
 		)
+		(property "Sim.Enable" ""
+			(at 177.8 107.95 0)
+			(hide yes)
+			(show_name no)
+			(do_not_autoplace no)
+			(effects
+				(font
+					(size 1.27 1.27)
+				)
+			)
+		)
 		(property "Sim.Pin" ""
 			(at 177.8 107.95 0)
@@
 			)
 		)
+		(property "Sim.Enable" ""
+			(at 177.8 140.97 0)
+			(hide yes)
+			(show_name no)
+			(do_not_autoplace no)
+			(effects
+				(font
+					(size 1.27 1.27)
+				)
+			)
+		)
 		(property "Sim.Pin" ""
 			(at 177.8 140.97 0)
@@
 			)
 		)
+		(property "Sim.Enable" ""
+			(at 177.8 125.73 0)
+			(hide yes)
+			(show_name no)
+			(do_not_autoplace no)
+			(effects
+				(font
+					(size 1.27 1.27)
+				)
+			)
+		)
 		(property "Sim.Pin" ""
 			(at 177.8 125.73 0)
@@
 			)
 		)
+		(property "Sim.Enable" ""
+			(at 177.8 90.17 0)
+			(hide yes)
+			(show_name no)
+			(do_not_autoplace no)
+			(effects
+				(font
+					(size 1.27 1.27)
+				)
+			)
+		)
 		(property "Sim.Pin" ""
 			(at 177.8 90.17 0)
@@
 			)
 		)
+		(property "Sim.Enable" ""
+			(at 177.8 144.78 0)
+			(hide yes)
+			(show_name no)
+			(do_not_autoplace no)
+			(effects
+				(font
+					(size 1.27 1.27)
+				)
+			)
+		)
 		(property "Sim.Pin" ""
 			(at 177.8 144.78 0)
@@
 			)
 		)
+		(property "Sim.Enable" ""
+			(at 177.8 93.98 0)
+			(hide yes)
+			(show_name no)
+			(do_not_autoplace no)
+			(effects
+				(font
+					(size 1.27 1.27)
+				)
+			)
+		)
 		(property "Sim.Pin" ""
 			(at 177.8 93.98 0)
@@
 		(in_pos_files no)
 		(dnp no)
-		(property "Reference" "#PWR0402"
+		(property "Reference" "#PWR402"
 			(at 146.05 62.23 0)
 			(hide yes)
@@
 			(project "beat-4"
 				(path "/6c8448b4-b04d-47e1-934e-e40cbe27a7be/a3f8c764-16c0-4eab-81c9-369dce0a6b86"
-					(reference "#PWR0402")
+					(reference "#PWR402")
 					(unit 1)
 				)
@@
 			)
 		)
+		(property "Sim.Enable" ""
+			(at 177.8 111.76 0)
+			(hide yes)
+			(show_name no)
+			(do_not_autoplace no)
+			(effects
+				(font
+					(size 1.27 1.27)
+				)
+			)
+		)
 		(property "Sim.Pin" ""
 			(at 177.8 111.76 0)
@@
 			)
 		)
+		(property "Sim.Enable" ""
+			(at 177.8 129.54 0)
+			(hide yes)
+			(show_name no)
+			(do_not_autoplace no)
+			(effects
+				(font
+					(size 1.27 1.27)
+				)
+			)
+		)
 		(property "Sim.Pin" ""
 			(at 177.8 129.54 0)
@@
 		(in_pos_files no)
 		(dnp no)
-		(property "Reference" "#PWR0401"
+		(property "Reference" "#PWR401"
 			(at 40.64 99.06 0)
 			(hide yes)
@@
 			(project "beat-4"
 				(path "/6c8448b4-b04d-47e1-934e-e40cbe27a7be/a3f8c764-16c0-4eab-81c9-369dce0a6b86"
-					(reference "#PWR0401")
+					(reference "#PWR401")
 					(unit 1)
 				)
@@
 			)
 		)
-		(property "Sheetfile" "PWMChannel.kicad_sch"
+		(property "Sheetfile" "PWM-Channel.kicad_sch"
 			(at 110.49 114.8846 0)
 			(hide yes)
@@
 			)
 		)
-		(property "Sheetfile" "PWMChannel.kicad_sch"
+		(property "Sheetfile" "PWM-Channel.kicad_sch"
 			(at 110.49 97.1046 0)
 			(hide yes)
@@
 			)
 		)
-		(property "Sheetfile" "PWMChannel.kicad_sch"
+		(property "Sheetfile" "PWM-Channel.kicad_sch"
 			(at 110.49 150.4446 0)
 			(hide yes)
@@
 			)
 		)
-		(property "Sheetfile" "PWMChannel.kicad_sch"
+		(property "Sheetfile" "PWM-Channel.kicad_sch"
 			(at 110.49 132.6646 0)
 			(hide yes)
@@
 			)
 		)
-		(property "Sheetfile" "PowerSwitch.kicad_sch"
+		(property "Sheetfile" "Power-Switch.kicad_sch"
 			(at 133.35 75.5146 0)
 			(hide yes)
